File: Macropad_STM32/Macropad_STM32.kicad_pcb (KiCad board)
At the start: 2 copper layers, 106 parts, among them J1 USB_C_Receptacle_USB2.0, J10 Encoders + LED, J2 Conn_01x04_Pin, J3 JTAG, J4 USB_C_Receptacle_USB2.0, J5 USB_C_Receptacle_USB2.0, J6 USB_C_Receptacle_USB2.0, J7 Power Connector, J9 Matrix, SW1 SW_Push, U1 STM32F103C8T6, U2 CY7C65632-28LTXCT, U3 AMS1117-3.3, U4 USBLC6-2SC6, U5 USBLC6-2SC6, U6 USBLC6-2SC6, U7 USBLC6-2SC6, Y1 16MHz, Y2 12MHz

Commit message: Matrix PCB layout done
Parts:
- added C39: 100n, Capacitor_SMD:C_0805_2012Metric_Pad1.18x1.45mm_HandSolder, F.Cu at (248.2, 65.7)
- added C40: 100n, Capacitor_SMD:C_0805_2012Metric_Pad1.18x1.45mm_HandSolder, F.Cu at (195.2, 66.0)
- added C41: 100n, Capacitor_SMD:C_0805_2012Metric_Pad1.18x1.45mm_HandSolder, F.Cu at (244.4, 65.7)
- added C42: 100n, Capacitor_SMD:C_0805_2012Metric_Pad1.18x1.45mm_HandSolder, F.Cu at (191.2, 66.0)
- added C43: 100n, Capacitor_SMD:C_0603_1608Metric_Pad1.08x0.95mm_HandSolder, F.Cu at (196.8, 91.0)
- added C44: 100n, Capacitor_SMD:C_0603_1608Metric_Pad1.08x0.95mm_HandSolder, F.Cu at (196.8, 107.2)
- added C45: 100n, Capacitor_SMD:C_0603_1608Metric_Pad1.08x0.95mm_HandSolder, F.Cu at (196.8, 122.8)
- added C46: 100n, Capacitor_SMD:C_0603_1608Metric_Pad1.08x0.95mm_HandSolder, F.Cu at (196.8, 138.7)
- added C47: 100n, Capacitor_SMD:C_0603_1608Metric_Pad1.08x0.95mm_HandSolder, F.Cu at (214.4, 91.0)
- added C48: 100n, Capacitor_SMD:C_0603_1608Metric_Pad1.08x0.95mm_HandSolder, F.Cu at (214.4, 107.0)
- added C49: 100n, Capacitor_SMD:C_0603_1608Metric_Pad1.08x0.95mm_HandSolder, F.Cu at (214.4, 122.8)
- added C50: 100n, Capacitor_SMD:C_0603_1608Metric_Pad1.08x0.95mm_HandSolder, F.Cu at (214.4, 138.7)
- added C51: 100n, Capacitor_SMD:C_0603_1608Metric_Pad1.08x0.95mm_HandSolder, F.Cu at (249.8, 91.0)
- added C52: 100n, Capacitor_SMD:C_0603_1608Metric_Pad1.08x0.95mm_HandSolder, F.Cu at (249.8, 107.0)
- added C53: 100n, Capacitor_SMD:C_0603_1608Metric_Pad1.08x0.95mm_HandSolder, F.Cu at (241.0, 126.2)
- added C54: 100n, Capacitor_SMD:C_0603_1608Metric_Pad1.08x0.95mm_HandSolder, F.Cu at (249.8, 138.7)
- added C55: 100n, Capacitor_SMD:C_0603_1608Metric_Pad1.08x0.95mm_HandSolder, F.Cu at (232.2, 91.0)
- added C56: 100n, Capacitor_SMD:C_0603_1608Metric_Pad1.08x0.95mm_HandSolder, F.Cu at (232.2, 107.0)
- added C57: 100n, Capacitor_SMD:C_0603_1608Metric_Pad1.08x0.95mm_HandSolder, F.Cu at (232.2, 122.8)
- added C58: 100n, Capacitor_SMD:C_0603_1608Metric_Pad1.08x0.95mm_HandSolder, F.Cu at (232.2, 138.7)
- added D13: 1N4148, Diode_SMD:D_SOD-123, F.Cu at (186.9, 87.0)
- added D14: 1N4148, Diode_SMD:D_SOD-123, F.Cu at (186.9, 102.8)
- added D15: 1N4148, Diode_SMD:D_SOD-123, F.Cu at (186.9, 118.8)
- added D16: 1N4148, Diode_SMD:D_SOD-123, F.Cu at (186.9, 134.7)
- added D17: 1N4148, Diode_SMD:D_SOD-123, F.Cu at (204.6, 87.0)
- added D18: 1N4148, Diode_SMD:D_SOD-123, F.Cu at (204.6, 102.8)
- added D19: 1N4148, Diode_SMD:D_SOD-123, F.Cu at (204.6, 118.8)
- added D20: 1N4148, Diode_SMD:D_SOD-123, F.Cu at (204.6, 134.7)
- added D21: 1N4148, Diode_SMD:D_SOD-123, F.Cu at (222.2, 87.0)
- added D22: 1N4148, Diode_SMD:D_SOD-123, F.Cu at (222.2, 102.8)
- added D23: 1N4148, Diode_SMD:D_SOD-123, F.Cu at (222.2, 118.8)
- added D24: 1N4148, Diode_SMD:D_SOD-123, F.Cu at (222.2, 134.7)
- added D25: 1N4148, Diode_SMD:D_SOD-123, F.Cu at (240.0, 87.0)
- added D26: 1N4148, Diode_SMD:D_SOD-123, F.Cu at (240.0, 102.8)
- added D27: 1N4148, Diode_SMD:D_SOD-123, F.Cu at (240.0, 118.8)
- added D28: 1N4148, Diode_SMD:D_SOD-123, F.Cu at (240.0, 134.7)
- added D29: SK6812MINI, KicadFootprints:SK6812-MINI-E, F.Cu at (193.3, 93.6)
- added D30: SK6812MINI, KicadFootprints:SK6812-MINI-E, F.Cu at (210.9, 93.6)
- added D31: SK6812MINI, KicadFootprints:SK6812-MINI-E, F.Cu at (228.7, 93.6)
- added D32: SK6812MINI, KicadFootprints:SK6812-MINI-E, F.Cu at (246.4, 93.6)
- added D33: SK6812MINI, KicadFootprints:SK6812-MINI-E, F.Cu at (193.3, 109.6)
- added D34: SK6812MINI, KicadFootprints:SK6812-MINI-E, F.Cu at (210.9, 109.6)
- added D35: SK6812MINI, KicadFootprints:SK6812-MINI-E, F.Cu at (228.7, 109.6)
- added D36: SK6812MINI, KicadFootprints:SK6812-MINI-E, F.Cu at (246.4, 109.6)
- added D37: SK6812MINI, KicadFootprints:SK6812-MINI-E, F.Cu at (193.3, 125.4)
- added D38: SK6812MINI, KicadFootprints:SK6812-MINI-E, F.Cu at (193.3, 141.2)
- added D39: SK6812MINI, KicadFootprints:SK6812-MINI-E, F.Cu at (210.9, 125.4)
- added D40: SK6812MINI, KicadFootprints:SK6812-MINI-E, F.Cu at (210.9, 141.2)
- added D41: SK6812MINI, KicadFootprints:SK6812-MINI-E, F.Cu at (228.7, 125.4)
- added D42: SK6812MINI, KicadFootprints:SK6812-MINI-E, F.Cu at (228.7, 141.2)
- added D43: SK6812MINI, KicadFootprints:SK6812-MINI-E, F.Cu at (246.4, 125.4)
- added D44: SK6812MINI, KicadFootprints:SK6812-MINI-E, F.Cu at (246.4, 141.2)
- added H5: MountingHole, MountingHole:MountingHole_3.2mm_M3_DIN965, F.Cu at (181.8, 61.6)
- added H6: MountingHole, MountingHole:MountingHole_3.2mm_M3_DIN965, F.Cu at (261.0, 61.6)
- added H7: MountingHole, MountingHole:MountingHole_3.2mm_M3_DIN965, F.Cu at (261.0, 141.6)
- added H8: MountingHole, MountingHole:MountingHole_3.2mm_M3_DIN965, F.Cu at (181.8, 141.6)
- added J11: Encoders + LED, Connector_JST:JST_EH_B7B-EH-A_1x07_P2.50mm_Vertical, F.Cu at (211.7, 76.0)
- added J12: Power Connector, Connector_JST:JST_EH_B3B-EH-A_1x03_P2.50mm_Vertical, F.Cu at (216.9, 63.5)
- added J8: Matrix, Connector_JST:JST_EH_B8B-EH-A_1x08_P2.50mm_Vertical, F.Cu at (181.8, 83.7)
- added K1: Kailh Hotswap Socket, KicadFootprints:Kailh_socket_MX_platemount, B.Cu at (193.3, 88.2)
- added K10: Kailh Hotswap Socket, KicadFootprints:Kailh_socket_MX_platemount, B.Cu at (228.6, 119.9)
- added K11: Kailh Hotswap Socket, KicadFootprints:Kailh_socket_MX_platemount, B.Cu at (228.6, 135.8)
- added K12: Kailh Hotswap Socket, KicadFootprints:Kailh_socket_MX_platemount, B.Cu at (228.7, 88.2)
- added K13: Kailh Hotswap Socket, KicadFootprints:Kailh_socket_MX_platemount, B.Cu at (246.4, 88.2)
- added K14: Kailh Hotswap Socket, KicadFootprints:Kailh_socket_MX_platemount, B.Cu at (246.4, 104.1)
- added K15: Kailh Hotswap Socket, KicadFootprints:Kailh_socket_MX_platemount, B.Cu at (246.4, 119.9)
- added K16: Kailh Hotswap Socket, KicadFootprints:Kailh_socket_MX_platemount, B.Cu at (246.4, 135.8)
- added K2: Kailh Hotswap Socket, KicadFootprints:Kailh_socket_MX_platemount, B.Cu at (193.3, 104.1)
- added K3: Kailh Hotswap Socket, KicadFootprints:Kailh_socket_MX_platemount, B.Cu at (193.3, 119.9)
- added K4: Kailh Hotswap Socket, KicadFootprints:Kailh_socket_MX_platemount, B.Cu at (193.3, 135.8)
- added K5: Kailh Hotswap Socket, KicadFootprints:Kailh_socket_MX_platemount, B.Cu at (211.0, 88.2)
- added K6: Kailh Hotswap Socket, KicadFootprints:Kailh_socket_MX_platemount, B.Cu at (211.0, 104.1)
- added K7: Kailh Hotswap Socket, KicadFootprints:Kailh_socket_MX_platemount, B.Cu at (211.0, 119.9)
- added K8: Kailh Hotswap Socket, KicadFootprints:Kailh_socket_MX_platemount, B.Cu at (211.0, 135.8)
- added K9: Kailh Hotswap Socket, KicadFootprints:Kailh_socket_MX_platemount, B.Cu at (228.6, 104.1)
- added R24: 10K, Resistor_SMD:R_0805_2012Metric_Pad1.20x1.40mm_HandSolder, F.Cu at (251.6, 73.5)
- added R25: 10K, Resistor_SMD:R_0805_2012Metric_Pad1.20x1.40mm_HandSolder, F.Cu at (198.4, 73.7)
- added R26: 500, Resistor_SMD:R_0805_2012Metric_Pad1.20x1.40mm_HandSolder, F.Cu at (252.6, 141.8)
- added R27: 500, Resistor_SMD:R_0805_2012Metric_Pad1.20x1.40mm_HandSolder, F.Cu at (187.6, 92.7)
- added R28: 10K, Resistor_SMD:R_0805_2012Metric_Pad1.20x1.40mm_HandSolder, F.Cu at (243.0, 61.6)
- added R29: 10K, Resistor_SMD:R_0805_2012Metric_Pad1.20x1.40mm_HandSolder, F.Cu at (251.0, 61.6)
- added R30: 10K, Resistor_SMD:R_0805_2012Metric_Pad1.20x1.40mm_HandSolder, F.Cu at (244.4, 63.6)
- added R31: 10K, Resistor_SMD:R_0805_2012Metric_Pad1.20x1.40mm_HandSolder, F.Cu at (248.2, 63.6)
- added R32: 10K, Resistor_SMD:R_0805_2012Metric_Pad1.20x1.40mm_HandSolder, F.Cu at (190.0, 62.0)
- added R33: 10K, Resistor_SMD:R_0805_2012Metric_Pad1.20x1.40mm_HandSolder, F.Cu at (197.8, 62.0)
- added R34: 10K, Resistor_SMD:R_0805_2012Metric_Pad1.20x1.40mm_HandSolder, F.Cu at (191.4, 64.0)
- added R35: 10K, Resistor_SMD:R_0805_2012Metric_Pad1.20x1.40mm_HandSolder, F.Cu at (195.2, 64.0)
- added SW2: EC11 Encoder, Rotary_Encoder:RotaryEncoder_Bourns_Vertical_PEC12R-3xxxF-Sxxxx, B.Cu at (244.5, 59.7)
- added SW3: EC11 Encoder, Rotary_Encoder:RotaryEncoder_Bourns_Vertical_PEC12R-3xxxF-Sxxxx, B.Cu at (191.4, 60.0)
- moved H1 99.0 mm to (128.2, 61.5)
- moved H2 99.0 mm to (128.2, 68.7)
- moved H3 99.0 mm to (128.2, 75.8)
- moved H4 99.0 mm to (128.2, 83.0)
- moved J4 88.4 mm to (112.8, 52.6)
- moved J5 88.4 mm to (112.8, 63.1)
- moved J6 88.4 mm to (112.8, 73.5)
- moved J2 69.6 mm to (119.2, 111.1)
- moved D10 58.7 mm to (44.3, 119.5)
- moved D11 58.7 mm to (44.3, 123.4)
- moved D2 58.7 mm to (32.1, 119.5)
- moved D3 58.7 mm to (32.1, 123.4)
- moved D6 58.7 mm to (38.2, 119.5)
- moved D7 58.7 mm to (38.2, 123.4)
- moved D1 58.7 mm to (32.1, 115.6)
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Other:
- board outline added: 255.9 x 163.3 mm

Commit message: Finished PCB layout, TODO: traces
Parts:
- removed C37: 100n, Capacitor_SMD:C_0805_2012Metric_Pad1.18x1.45mm_HandSolder
- removed D11: SK6812, SK6812SIDE:SK6812SIDE
- removed FB4: 600R, Fuse:Fuse_0805_2012Metric_Pad1.15x1.40mm_HandSolder
- removed R18, R19, R20, R21: 10k, Resistor_SMD:R_0805_2012Metric_Pad1.20x1.40mm_HandSolder
- added FB5: 600R, Fuse:Fuse_0805_2012Metric_Pad1.15x1.40mm_HandSolder, F.Cu at (76.0, 30.7)
- moved C39 145.6 mm to (106.2, 97.6)
- moved C40 145.6 mm to (53.2, 98.0)
- moved C42 145.6 mm to (49.2, 98.0)
- moved C43 145.6 mm to (54.8, 123.0)
- moved C44 145.6 mm to (54.8, 139.2)
- moved C45 145.6 mm to (54.8, 154.8)
- moved C46 145.6 mm to (54.8, 170.6)
- moved C51 145.6 mm to (107.8, 123.0)
- moved C52 145.6 mm to (107.8, 139.0)
- moved C54 145.6 mm to (107.8, 170.6)
- moved C55 145.6 mm to (90.2, 123.0)
- moved C56 145.6 mm to (90.2, 139.0)
- moved C57 145.6 mm to (90.2, 154.8)
- moved C58 145.6 mm to (90.2, 170.6)
- moved D21 145.6 mm to (80.2, 119.0)
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Connections:
- C9 pad 1: /NRST_SW_C -> /NRST
- D12 pad 1: Net-(D11-DOUT) -> Net-(D10-DOUT)
- FB2 pad 1: Net-(F2-Pad2) -> Net-(F3-Pad2)
- FB2 pad 2: +5V -> VBUS
- FB3 pad 1: Net-(F3-Pad2) -> Net-(F4-Pad2)
- FB3 pad 2: +5V -> VBUS
- J3 pad 9: /SWCLK -> /SWDIO
- R1 pad 2: /NRST_SW_C -> /NRST
- R14 pad 2: +3.3V -> /NRST
- SW1 pad 1: /NRST_SW_C -> /NRST
- U1 pad 7: +3.3V -> /NRST
Other:
- board size 255.9 x 163.3 mm -> 98 x 159.1 mm

Commit message: Schematic changes Motherboard nearing completion
Parts:
- removed F2: 500mA, Fuse:Fuse_1206_3216Metric_Pad1.42x1.75mm_HandSolder
- removed FB5: 600R, Fuse:Fuse_0805_2012Metric_Pad1.15x1.40mm_HandSolder
- removed J11: Encoders + LED, Connector_JST:JST_EH_B7B-EH-A_1x07_P2.50mm_Vertical
- removed J8: Matrix, Connector_JST:JST_EH_B8B-EH-A_1x08_P2.50mm_Vertical
- removed U5: USBLC6-2SC6, Package_TO_SOT_SMD:SOT-23-6
- added C37: 2u2, Capacitor_SMD:C_0805_2012Metric_Pad1.18x1.45mm_HandSolder, F.Cu at (52.3, 74.9)
- added C59: 2u2, Capacitor_SMD:C_0805_2012Metric_Pad1.18x1.45mm_HandSolder, F.Cu at (52.3, 77.9)
- added C61: 100u, Capacitor_SMD:C_Elec_6.3x5.4, F.Cu at (45.0, 82.6)
- added C62: 100u, Capacitor_SMD:C_Elec_6.3x5.4, F.Cu at (45.0, 90.7)
- added D11: SK6812, SK6812SIDE:SK6812SIDE, F.Cu at (94.1, 63.5)
- added F5: 500mA, Fuse:Fuse_1206_3216Metric_Pad1.42x1.75mm_HandSolder, F.Cu at (62.9, 75.3)
- added FB4: 120R, Fuse:Fuse_0805_2012Metric_Pad1.15x1.40mm_HandSolder, F.Cu at (52.3, 83.8)
- added J13: Conn_01x04_Socket, Connector_PinHeader_2.54mm:PinHeader_1x04_P2.54mm_Vertical, F.Cu at (114.6, 68.1)
- added J14: Conn_01x04_Socket, Connector_PinHeader_2.54mm:PinHeader_1x04_P2.54mm_Vertical, F.Cu at (51.6, 60.4)
- added J15: USB_C_Receptacle_USB2.0, Connector_USB:USB_C_Receptacle_HRO_TYPE-C-31-M-12, F.Cu at (34.1, 74.4)
- added J16: Conn_01x04_Socket, Connector_PinHeader_2.54mm:PinHeader_1x04_P2.54mm_Vertical, F.Cu at (145.0, 55.6)
- added J17: Conn_01x04_Socket, Connector_PinHeader_2.54mm:PinHeader_1x04_P2.54mm_Vertical, F.Cu at (56.3, 60.4)
- added J18: Conn_01x04_Socket, Connector_PinHeader_2.54mm:PinHeader_1x04_P2.54mm_Vertical, F.Cu at (132.6, 55.6)
- added J19: Conn_01x04_Socket, Connector_PinHeader_2.54mm:PinHeader_1x04_P2.54mm_Vertical, F.Cu at (109.2, 37.3)
- added J20: USB_C_Receptacle_USB2.0, Connector_USB:USB_C_Receptacle_HRO_TYPE-C-31-M-12, F.Cu at (34.1, 84.8)
- added J21: Matrix, Connector_JST:JST_EH_B8B-EH-A_1x08_P2.50mm_Vertical, F.Cu at (-89.4, 116.0)
- added J22: Encoders + LED, Connector_JST:JST_EH_B7B-EH-A_1x07_P2.50mm_Vertical, F.Cu at (-109.9, 101.3)
- added U8: USBLC6-2SC6, Package_TO_SOT_SMD:SOT-23-6, F.Cu at (57.3, 77.0)
- C18: value 100n -> 2u2
- C19: value 100n -> 100u; footprint Capacitor_SMD:C_0805_2012Metric_Pad1.18x1.45mm_HandSolder -> Capacitor_SMD:C_Elec_6.3x5.4
- C24: value 100n -> locked
- FB2, FB3: value 600R -> 120R
- J4, J5: value USB_C_Receptacle_USB2.0 -> Conn_01x04_Socket; footprint Connector_USB:USB_C_Receptacle_HRO_TYPE-C-31-M-12 -> Connector_PinHeader_2.54mm:PinHeader_1x04_P2.54mm_Vertical
- moved C39 186.4 mm to (-75.8, 137.7)
- moved C40 186.4 mm to (-128.8, 138.1)
- moved C41 186.4 mm to (-79.6, 137.7)
- moved C42 186.4 mm to (-132.8, 138.1)
- moved C43 186.4 mm to (-127.2, 163.1)
- moved C44 186.4 mm to (-127.2, 179.3)
- moved C45 186.4 mm to (-127.2, 194.9)
- moved C46 186.4 mm to (-127.2, 210.7)
- moved C47 186.4 mm to (-109.6, 163.1)
- moved C48 186.4 mm to (-109.6, 179.1)
- moved C49 186.4 mm to (-109.6, 194.9)
- moved C50 186.4 mm to (-109.6, 210.7)
- moved C51 186.4 mm to (-74.2, 163.1)
- moved C52 186.4 mm to (-74.2, 179.1)
- moved C53 186.4 mm to (-83.0, 198.3)
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Connections:
- C12 pad 2: VBUS -> /VBUS_IN
- C17 pad 1: Net-(U5-VBUS) -> VBUS
- C18 pad 1: Net-(U6-VBUS) -> Net-(J17-Pin_1)
- C19 pad 1: Net-(U7-VBUS) -> Net-(C19-Pad1)
- D12 pad 1: Net-(D10-DOUT) -> Net-(D11-DOUT)
- F1 pad 2: VBUS -> /VBUS_IN
- F3 pad 1: Net-(U6-VBUS) -> /USBHUB/D1_VBUS
- F4 pad 1: Net-(U7-VBUS) -> /USBHUB/D3_VBUS
- FB2 pad 2: VBUS -> Net-(J19-Pin_1)
- FB3 pad 2: VBUS -> Net-(J14-Pin_1)
- J1 pad A1: GND -> /USB_UP_GND
- J1 pad A12: GND -> /USB_UP_GND
- J1 pad B1: GND -> /USB_UP_GND
- J1 pad B12: GND -> /USB_UP_GND
- J1 pad S1: GND -> /USB_UP_GND
- J6 pad A1: GND -> /USBHUB/D3_GND
- J6 pad A12: GND -> /USBHUB/D3_GND
- J6 pad A4: Net-(U7-VBUS) -> /USBHUB/D3_VBUS
- J6 pad A9: Net-(U7-VBUS) -> /USBHUB/D3_VBUS
- J6 pad B1: GND -> /USBHUB/D3_GND
- J6 pad B12: GND -> /USBHUB/D3_GND
- J6 pad B4: Net-(U7-VBUS) -> /USBHUB/D3_VBUS
- J6 pad B9: Net-(U7-VBUS) -> /USBHUB/D3_VBUS
- J6 pad S1: GND -> /USBHUB/D3_GND
- K10 pad 1: /Matrix/COL1 -> /Matrix/COL2
- K11 pad 1: /Matrix/COL1 -> /Matrix/COL2
- K12 pad 1: /Matrix/COL1 -> /Matrix/COL2
- K13 pad 1: /Matrix/COL0 -> /Matrix/COL3
- K14 pad 1: /Matrix/COL0 -> /Matrix/COL3
- K15 pad 1: /Matrix/COL0 -> /Matrix/COL3
- K16 pad 1: /Matrix/COL0 -> /Matrix/COL3
- K9 pad 1: /Matrix/COL1 -> /Matrix/COL2
- U1 pad 2: unconnected-(U1-PC13-Pad2) -> /LED
- U1 pad 45: /LED -> unconnected-(U1-PB8-Pad45)
- U2 pad 1: /USBHUB/UP_USB_D- -> /UP_USB_D-
- U2 pad 2: /USBHUB/UP_USB_D+ -> /UP_USB_D+
- U4 pad 1: /USBHUB/UP_USB_D- -> /UP_USB_D-
- U4 pad 2: GND -> /USB_UP_GND
- U4 pad 3: /USBHUB/UP_USB_D+ -> /UP_USB_D+
- U4 pad 5: +3.3V -> /VBUS_IN
- U6 pad 1: Net-(J5-D--PadA7) -> Net-(J15-D--PadA7)
- U6 pad 2: GND -> /USBHUB/D2_GND
- U6 pad 3: Net-(J5-D+-PadA6) -> Net-(J15-D+-PadA6)
- U6 pad 5: Net-(U6-VBUS) -> /USBHUB/D2_VBUS
- U7 pad 2: GND -> /USBHUB/D3_GND
- U7 pad 5: Net-(U7-VBUS) -> /USBHUB/D3_VBUS
Routing:
- net /NRST: track 0.00 -> 58.6 mm, vias 0 -> 2
- net /SWDIO: track 0.00 -> 47.1 mm
- net /SWO: track 0.00 -> 46.0 mm
- net /SWCLK: track 0.00 -> 42.0 mm
- net /ENC2_SW: track 0.00 -> 35.7 mm
- net /UP_USB_D+: track 0.00 -> 34.0 mm
- net /UP_USB_D-: track 0.00 -> 33.9 mm
- net /TDI: track 0.00 -> 33.8 mm
- net /ENC2_B: track 0.00 -> 33.1 mm
- net /tRST: track 0.00 -> 31.9 mm
- net /Key_LED: track 0.00 -> 31.5 mm, vias 0 -> 2
- net /USBHUB/D2_D-: track 0.00 -> 31.1 mm
- net /ENC2_A: track 0.00 -> 30.4 mm
- net /USBHUB/D2_D+: track 0.00 -> 30.3 mm
- net /ENC1_SW: track 0.00 -> 28.0 mm
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Other:
- board size 98 x 159.1 mm -> 340.3 x 176.3 mm
- copper layers 2 -> 4
- rule pad_to_mask_clearance: 0 -> 0.038

Commit message: Minor changes to motherboard
Parts:
- moved H7 88.2 mm to (-27.5, 132.9)
- moved H8 88.2 mm to (-106.7, 132.9)
- moved R26 88.2 mm to (-35.9, 133.2)
- moved C44 88.2 mm to (-91.7, 98.6)
- moved C45 88.2 mm to (-91.7, 114.2)
- moved C49 88.2 mm to (-74.1, 114.2)
- moved C53 88.2 mm to (-47.5, 117.6)
- moved C57 88.2 mm to (-56.3, 114.2)
- moved D13 88.2 mm to (-101.6, 78.3)
- moved D14 88.2 mm to (-101.6, 94.2)
- moved D18 88.2 mm to (-83.9, 94.2)
- moved D19 88.2 mm to (-83.9, 110.2)
- moved D22 88.2 mm to (-66.3, 94.2)
- moved D23 88.2 mm to (-66.3, 110.2)
- moved D26 88.2 mm to (-48.5, 94.2)
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Routing:
- net /SWCLK: track 42.0 -> 29.8 mm
- net /SWDIO: track 47.1 -> 35.2 mm
- net /NRST: track 58.6 -> 70.4 mm
- net /TDI: track 33.8 -> 26.6 mm
- net /USBHUB/D2_D+: track 30.3 -> 23.5 mm
- net /USBHUB/D2_D-: track 31.1 -> 24.5 mm
- net /SWO: track 46.0 -> 39.6 mm
- net /USBHUB/D3_D-: track 23.8 -> 17.6 mm
- net /tRST: track 31.9 -> 25.8 mm
- net /USBHUB/D3_D+: track 23.7 -> 17.6 mm
- net /JP_BOOT0: track 10.3 -> 9.44 mm
Other:
- board size 340.3 x 176.3 mm -> 304.7 x 95.5 mm

Commit message: Revision 1 nearly finished
Parts:
- removed J15, J20: USB_C_Receptacle_USB2.0, Connector_USB:USB_C_Receptacle_HRO_TYPE-C-31-M-12
- added H11: MountingHole, MountingHole:MountingHole_2.2mm_M2, F.Cu at (78.3, 125.6)
- added H12: MountingHole, MountingHole:MountingHole_2.2mm_M2, F.Cu at (78.3, 100.2)
- added H13: MountingHole, MountingHole:MountingHole_2.2mm_M2, F.Cu at (78.4, 74.6)
- added H14: MountingHole, MountingHole:MountingHole_2.2mm_M2, F.Cu at (78.4, 93.0)
- added H15: MountingHole, MountingHole:MountingHole_2.2mm_M2, F.Cu at (133.7, 66.2)
- added H15: MountingHole, MountingHole:MountingHole_2.2mm_M2, F.Cu at (99.5, 66.2)
- added H16: MountingHole, MountingHole:MountingHole_2.2mm_M2, F.Cu at (151.4, 53.3)
- added H16: MountingHole, MountingHole:MountingHole_2.2mm_M2, F.Cu at (117.1, 53.3)
- added J8: USB_A, SK6812SIDE:AMPHENOL_UE27AC54100, F.Cu at (106.1, 61.1)
- C17, C20, C21, C29, C30, C31, C32, C33, C34, C35, C36, C38, C39, C40, C41, C42, D1, D10, D11, D12, D2, D3, D4, D5, D6, D7, D8, D9, R22, R23, R24, R25, R28, R29, R30, R31, R32, R33, R34, R35: moved to B.Cu
- J13, J14, J16, J17, J18, J19, J4, J5: footprint Connector_PinHeader_2.54mm:PinHeader_1x04_P2.54mm_Vertical -> SK6812SIDE:MOLEX_0781710004
- J2: value Conn_01x04_Pin -> USB_A; footprint Connector_PinHeader_2.54mm:PinHeader_1x04_P2.54mm_Vertical -> SK6812SIDE:AMPHENOL_UE27AC54100
- SW2, SW3: moved to F.Cu
- moved R32 290.4 mm to (192.0, 57.0), turned to 180 degrees
- moved R28 290.1 mm to (244.6, 56.6), turned to 0 degrees
- moved C53 290.0 mm to (242.6, 117.8), turned to 0 degrees
- moved C42 288.0 mm to (190.8, 61.0), turned to 0 degrees
- moved SW3 287.7 mm to (190.6, 54.9)
- moved R34 287.6 mm to (190.6, 59.0), turned to 180 degrees
- moved C41 287.3 mm to (243.2, 60.6), turned to 0 degrees
- moved R30 287.3 mm to (243.2, 58.6), turned to 180 degrees
- moved SW2 287.1 mm to (243.1, 54.7)
- moved J21 281.9 mm to (173.8, 74.9), turned to -90 degrees
- moved C43 281.1 mm to (189.4, 86.0)
- moved C44 281.1 mm to (189.4, 102.2)
- moved C45 281.1 mm to (189.4, 117.8)
- moved C46 281.1 mm to (189.4, 133.6)
- moved C47 281.1 mm to (207.0, 86.0)
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Connections:
- C12 pad 1: GND -> /USB_UP_GND
- C18 pad 2: GND -> /USBHUB/D2_GND
- C19 pad 2: GND -> /USBHUB/D2_GND
- C27 pad 1: +3V3 -> +3.3V
- C28 pad 1: +3V3 -> +3.3V
- C37 pad 2: GND -> /USBHUB/D1_GND
- C39 pad 1: /Matrix/ENC_1_B -> /Matrix/ENC_1_A
- C39 pad 2: GND -> GND1
- C40 pad 1: /Matrix/ENC_2_B -> /Matrix/ENC_2_A
- C40 pad 2: GND -> GND1
- C41 pad 2: GND -> GND1
- C42 pad 2: GND -> GND1
- C43 pad 1: VBUS -> +5V
- C43 pad 2: GND -> Net-(C43-Pad2)
- C44 pad 1: VBUS -> +5V
- C44 pad 2: GND -> GND1
- C45 pad 1: VBUS -> +5V
- C45 pad 2: GND -> GND1
- C46 pad 1: VBUS -> +5V
- C46 pad 2: GND -> Net-(C43-Pad2)
- C47 pad 1: VBUS -> +5V
- C47 pad 2: GND -> GND1
- C48 pad 1: VBUS -> +5V
- C48 pad 2: GND -> GND1
- C49 pad 1: VBUS -> +5V
- C49 pad 2: GND -> Net-(C43-Pad2)
- C50 pad 1: VBUS -> +5V
- C50 pad 2: GND -> GND1
- C51 pad 1: VBUS -> +5V
- C51 pad 2: GND -> GND1
- C52 pad 1: VBUS -> +5V
- C52 pad 2: GND -> Net-(C43-Pad2)
- C53 pad 1: VBUS -> +5V
- C53 pad 2: GND -> GND1
- C54 pad 1: VBUS -> +5V
- C54 pad 2: GND -> GND1
- C55 pad 1: VBUS -> +5V
- C55 pad 2: GND -> GND1
- C56 pad 1: VBUS -> +5V
- C56 pad 2: GND -> GND1
- C57 pad 1: VBUS -> +5V
- C57 pad 2: GND -> GND1
- C58 pad 1: VBUS -> +5V
- C58 pad 2: GND -> GND1
- C59 pad 2: GND -> /USBHUB/D3_GND
- C61 pad 2: GND -> /USBHUB/D1_GND
- C62 pad 2: GND -> /USBHUB/D3_GND
- D29 pad 1: VBUS -> +5V
- D29 pad 3: GND -> GND1
- D30 pad 1: VBUS -> +5V
- D30 pad 3: GND -> GND1
- D31 pad 1: VBUS -> +5V
- D31 pad 3: GND -> GND1
- D32 pad 1: VBUS -> +5V
- D32 pad 3: GND -> GND1
- D33 pad 1: VBUS -> +5V
- D33 pad 3: GND -> GND1
- D34 pad 1: VBUS -> +5V
- D34 pad 3: GND -> GND1
- D35 pad 1: VBUS -> +5V
- D35 pad 3: GND -> GND1
- D36 pad 1: VBUS -> +5V
- D36 pad 3: GND -> GND1
- D37 pad 1: VBUS -> +5V
- D37 pad 3: GND -> GND1
- D38 pad 1: VBUS -> +5V
- D38 pad 3: GND -> GND1
- D39 pad 1: VBUS -> +5V
- D39 pad 3: GND -> GND1
- D40 pad 1: VBUS -> +5V
- D40 pad 3: GND -> GND1
- D41 pad 1: VBUS -> +5V
- D41 pad 3: GND -> GND1
- D42 pad 1: VBUS -> +5V
- D42 pad 3: GND -> GND1
- D43 pad 1: VBUS -> +5V
- D43 pad 3: GND -> GND1
- D44 pad 1: VBUS -> +5V
- D44 pad 3: GND -> GND1
- J12 pad 1: VBUS -> +5V
- J12 pad 2: +3.3V -> +3V3
- J12 pad 3: GND -> GND1
- J14 pad 2: /USBHUB/D3_D- -> /USBHUB/Daughter_D3_D-
- J14 pad 3: /USBHUB/D3_D+ -> /USBHUB/Daughter_D3_D+
- J17 pad 2: /USBHUB/D2_D- -> /USBHUB/Daughter_D2_D-
- J17 pad 3: /USBHUB/D2_D+ -> /USBHUB/Daughter_D2_D+
- J19 pad 2: /USBHUB/D1_D- -> /USBHUB/Daughter_D1_D-
- J19 pad 3: /USBHUB/D1_D+ -> /USBHUB/Daughter_D1_D+
- J2 pad 1: +3.3V -> /USBHUB/D1_VBUS
- J2 pad 2: /SWDIO -> Net-(J2-D-)
- J2 pad 3: /SWCLK -> Net-(J2-D+)
- J2 pad 4: GND -> /USBHUB/D1_GND
- J21 pad 1: /Matrix/COL0 -> /Matrix/COL3
- J21 pad 2: /Matrix/COL1 -> /Matrix/COL2
- J21 pad 3: /Matrix/COL2 -> /Matrix/COL1
- J21 pad 4: /Matrix/COL3 -> /Matrix/COL0
- J22 pad 1: /Matrix/Key_LED -> +5V
- J22 pad 3: /Matrix/ENC_1_B -> /Matrix/ENC_1_A
- J22 pad 6: /Matrix/ENC_2_B -> /Matrix/ENC_2_A
- J9 pad 1: /COL0 -> /COL3
- J9 pad 2: /COL1 -> /COL2
- J9 pad 3: /COL2 -> /COL1
- J9 pad 4: /COL3 -> /COL0
- R24 pad 1: GND -> GND1
- R25 pad 1: GND -> GND1
- R26 pad 2: GND -> GND1
- R27 pad 1: /Matrix/Key_LED -> +5V
- R28 pad 2: +3.3V -> +3V3
- R29 pad 1: +3.3V -> +3V3
- R3 pad 2: GND -> /USB_UP_GND
- R31 pad 2: /Matrix/ENC_1_B -> /Matrix/ENC_1_A
- R32 pad 1: +3.3V -> +3V3
- R33 pad 1: +3.3V -> +3V3
- R35 pad 2: /Matrix/ENC_2_B -> /Matrix/ENC_2_A
- R4 pad 2: GND -> /USB_UP_GND
- SW2 pad C: GND -> GND1
- SW2 pad S1: +3.3V -> +3V3
- SW3 pad C: GND -> GND1
- SW3 pad S1: +3.3V -> +3V3
- U1 pad 10: /COL0 -> /COL3
- U1 pad 11: /COL1 -> /COL2
- U1 pad 12: /COL2 -> /COL1
- U1 pad 13: /COL3 -> /COL0
- U1 pad 18: unconnected-(U1-PB0-Pad18) -> /Key_LED
- U1 pad 46: /Key_LED -> unconnected-(U1-PB9-Pad46)
- U6 pad 4: /USBHUB/D2_D+ -> /USBHUB/Daughter_D2_D+
- U6 pad 6: /USBHUB/D2_D- -> /USBHUB/Daughter_D2_D-
- U7 pad 4: /USBHUB/D3_D+ -> /USBHUB/Daughter_D3_D+
- U7 pad 6: /USBHUB/D3_D- -> /USBHUB/Daughter_D3_D-
- U8 pad 1: Net-(J20-D--PadA7) -> Net-(J2-D-)
- U8 pad 3: Net-(J20-D+-PadA6) -> Net-(J2-D+)
- U8 pad 4: /USBHUB/D1_D+ -> /USBHUB/Daughter_D1_D+
- U8 pad 6: /USBHUB/D1_D- -> /USBHUB/Daughter_D1_D-
Routing:
- net +5V: track 0.00 -> 129.5 mm, vias 0 -> 16
- net /Matrix/COL3: track 0.00 -> 126.0 mm
- net /Matrix/COL2: track 0.00 -> 107.5 mm, vias 0 -> 6
- net /Matrix/ROW3: track 0.00 -> 99.1 mm
- net GND: track 4.48 -> 96.0 mm, vias 0 -> 33
- net /Matrix/COL1: track 0.00 -> 91.2 mm, vias 0 -> 6
- net /Matrix/ROW2: track 0.00 -> 85.6 mm
- net /Matrix/COL0: track 0.00 -> 77.9 mm, vias 0 -> 6
- net /Matrix/ROW1: track 0.00 -> 72.5 mm
- net /Matrix/LED89: track 0.00 -> 69.0 mm, vias 0 -> 2
- net /Matrix/LED45: track 0.00 -> 69.0 mm, vias 0 -> 2
- net /Matrix/LED1213: track 0.00 -> 68.3 mm, vias 0 -> 2
- net /Matrix/ROW0: track 0.00 -> 64.0 mm
- net /Matrix/ENC_1_A: track 0.00 -> 59.9 mm
- net /Matrix/ENC_2_A: track 0.00 -> 49.3 mm
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- added copper zone on F.Cu, net +3.3V
- added copper zone on In2.Cu, net +3.3V
- added copper zone on B.Cu, net +3.3VA
- added copper zone on F.Cu, net +3.3VA
- added copper zone on In2.Cu, net +3V3
- added copper zone on B.Cu, net +5V
- added copper zone on B.Cu, net /USBHUB/D1_GND
- added copper zone on F.Cu, net /USBHUB/D1_GND
- added copper zone on In1.Cu, net /USBHUB/D1_GND
- added copper zone on B.Cu, net /USBHUB/D1_VBUS
- added copper zone on In2.Cu, net /USBHUB/D1_VBUS
- added copper zone on B.Cu, net /USBHUB/D2_GND
- added copper zone on F.Cu, net /USBHUB/D2_GND
- added copper zone on In1.Cu, net /USBHUB/D2_GND
- added copper zone on In2.Cu, net /USBHUB/D2_VBUS
- added copper zone on B.Cu, net /USBHUB/D3_GND
- added copper zone on F.Cu, net /USBHUB/D3_GND
- added copper zone on In1.Cu, net /USBHUB/D3_GND
- added copper zone on In2.Cu, net /USBHUB/D3_VBUS
- added copper zone on B.Cu, net /USB_UP_GND
- added copper zone on F.Cu, net /USB_UP_GND
- added copper zone on In1.Cu, net /USB_UP_GND
- added copper zone on In2.Cu, net /VBUS_IN
- added copper zone on F.Cu, net GND
- added copper zone on In1.Cu, net GND
- added copper zone on F.Cu, net GND1
- added copper zone on In1.Cu, net GND1
- added copper zone on B.Cu, net VBUS
- added copper zone on F.Cu, net VBUS
Other:
- board size 304.7 x 95.5 mm -> 183.3 x 93.4 mm
